Commit message: added collision mesh to comau to prevent unexpected movement
added base orientation to initial rooting constraint

File: src/wbk_sim/robot_descriptions/comau_NJ290_3-0_m.urdf (robot description, URDF)
Before this commit: robot example_robot, 21 links, 20 joints
Links:
- link link0_passive: geometry collision mesh filename=mesh/base_m.stl; visual mesh filename=mesh/base_m.stl
- link link1_x_axis: geometry collision mesh filename=mesh/q1_m.stl; visual mesh filename=mesh/q1_m.stl
- link link2_x_axis: geometry collision mesh filename=mesh/q2_m.stl; visual mesh filename=mesh/q2_m.stl
- link link3_x_axis: geometry collision mesh filename=mesh/q3_m.stl; visual mesh filename=mesh/q3_m.stl
- link link4_x_axis: geometry collision mesh filename=mesh/q4_m.stl; visual mesh filename=mesh/q4_m.stl
- link link5_x_axis: geometry collision mesh filename=mesh/q5_m.stl; visual mesh filename=mesh/q5_m.stl
- link link6_x_axis: geometry collision mesh filename=mesh/q6_m.stl; visual mesh filename=mesh/q6_m.stl
