Commit message: fixed urdf so mill end coincides with tcp

File: examples/robot_descriptions/milling_head.urdf (robot description, URDF)
Before this commit: robot milling_head, 2 links, 1 joints
Links:
- removed link tcp_link
- added link tcp; visual cylinder length=0.50 radius=0.02
Joints:
- joint milling_trafo: child camera_frame -> tcp; origin xyz=0.5 0.0 0 rpy=0 1.57075 0 -> xyz=0.25 0.0 0 rpy=0 1.57075 0

Commit message: more stable base orientation calculation
also updated urdf for more predictable orientation behavior

File: examples/robot_descriptions/milling_head.urdf (robot description, URDF)
Before this commit: robot milling_head, 2 links, 1 joints
Links:
- link baseLink: geometry visual box size=0.15 0.15 0.3
Joints:
- joint milling_trafo: origin xyz=0.25 0.0 0 rpy=0 1.57075 0 -> xyz=0.3 0.0 0.0 rpy=0 -1.57075 0

Commit message: adjusted milling head visuals

File: examples/robot_descriptions/milling_head.urdf (robot description, URDF)
Before this commit: robot milling_head, 2 links, 1 joints
Links:
- link baseLink: geometry visual box size=0.3 0.15 0.15

Commit message: streamlined relative pose and orientation calculation, offset milling tool

File: examples/robot_descriptions/milling_head.urdf (robot description, URDF)
Before this commit: robot milling_head, 2 links, 1 joints
Joints:
- joint milling_trafo: origin xyz=0.3 0.0 0.0 rpy=0 -1.57075 0 -> xyz=0.3 0.0 0.1 rpy=0 -1.57075 0
