Commit message: working example for gripping

File: examples/robot_descriptions/gripper.urdf (robot description, URDF)
Before this commit: robot gripper, 4 links, 3 joints
Links:
- link baseLink: geometry collision box size=0.3 0.15 0.15; visual box size=0.3 0.15 0.15
Joints:
- joint finger_joint1: limit lower=0.0 upper=0.1 effort=20 velocity=0.2 -> lower=0.0 upper=0.11 effort=20 velocity=0.2
- joint finger_joint2: limit lower=-0 upper=0.1 effort=20 velocity=0.2 -> lower=-0 upper=0.11 effort=20 velocity=0.2
