Commit message: Implemented CAD-Gripper

File: examples/robot_descriptions/cube_small.urdf (robot description, URDF)
Before this commit: robot cube, 1 links, 0 joints
Links:
- link baseLink: mass 1.0 -> 0.1

File: examples/robot_descriptions/gripper_cad.urdf (robot description, URDF)
Before this commit: robot gripper, 4 links, 3 joints
Links:
- link baseLink: geometry visual mesh filename=tool_mesh/base_m.stl
- link leftfinger: geometry collision mesh filename=tool_mesh/finger01_m.stl; visual mesh filename=tool_mesh/finger01_m.stl
- link rightfinger: geometry collision mesh filename=tool_mesh/finger02_m.stl; visual mesh filename=tool_mesh/finger02_m.stl
Joints:
- joint finger_joint1: axis 0 0 1 -> -1 0 0; limit lower=0.0 upper=0.11 effort=200 velocity=0.2 -> lower=0.0 upper=0.11 effort=20 velocity=0.2; origin xyz=0.15 0 0.15 rpy=0 -1.57079632679 0 -> xyz=0.0 0 0.0 rpy=0 0 0
- joint finger_joint2: axis 0 0 -1 -> 1 0 0; limit lower=-0 upper=0.11 effort=200 velocity=0.2 -> lower=-0 upper=0.11 effort=20 velocity=0.2; origin xyz=-0.15 0 0.15 rpy=0 -1.57079632679 0 -> xyz=0.0 0 0.0 rpy=0 0 0
- joint gripping_trafo: origin xyz=0 0.0 0.25 rpy=0 0 0 -> xyz=0 0.0 0.39 rpy=0 0 0
