Commit message: implemented gripper, bugfix relative tcp positon

File: examples/robot_descriptions/gripper_cylinder.urdf (robot description, URDF)
Before this commit: robot gripper, 4 links, 3 joints
Links:
- link baseLink: geometry collision box size=0.3 0.15 0.15; visual box size=0.3 0.15 0.15
- link leftfinger: geometry collision cylinder length=0.2 radius=0.025; visual cylinder length=0.2 radius=0.025
- link rightfinger: geometry collision cylinder length=0.2 radius=0.025; visual cylinder length=0.2 radius=0.025
Joints:
- joint finger_joint1: limit lower=-0.05 upper=0.11 effort=20 velocity=0.2 -> lower=0.0 upper=0.11 effort=200 velocity=0.2; origin xyz=0.0 0 0.0 rpy=0 0 0 -> xyz=0.15 0 0.15 rpy=0 0 0
- joint finger_joint2: limit lower=-0.05 upper=0.11 effort=20 velocity=0.2 -> lower=-0 upper=0.11 effort=200 velocity=0.2; origin xyz=0.0 0 0.0 rpy=0 0 0 -> xyz=-0.15 0 0.15 rpy=0 0 0
- joint gripping_trafo: origin xyz=0 0.0 0.39 rpy=0 0 0 -> xyz=0 0.0 0.25 rpy=0 0 0
