Commit message: fixed tcp pose of 3d printing head

File: examples/robot_descriptions/3d_printing_head.urdf (robot description, URDF)
Before this commit: robot 3d_printing_head, 3 links, 2 joints
Links:
- removed link MDPH2
- link baseLink: geometry visual mesh filename=kuka_meshes/MDPH2.stl scale=0.001 0.001 0.001
- link tcp: geometry visual cylinder length=0.01 radius=0.001
Joints:
- removed joint Extruder
- removed joint z_rotation
- added joint milling_trafo: type fixed, parent baseLink, child tcp, origin xyz=-0.222558 0.1736378 0.0 rpy=0 1.57075 0
