Commit message: added kuka stl model and 3d printing head

File: examples/robot_descriptions/comau_NJ290_3-0_m.urdf (robot description, URDF)
Before this commit: robot example_robot, 21 links, 20 joints
Links:
- link link0_passive: geometry collision mesh filename=comau_meshes/base_m.stl; visual mesh filename=comau_meshes/base_m.stl
- link link1_x_axis: geometry collision mesh filename=comau_meshes/q1_m.stl; visual mesh filename=comau_meshes/q1_m.stl
- link link2_x_axis: geometry collision mesh filename=comau_meshes/q2_m.stl; visual mesh filename=comau_meshes/q2_m.stl
- link link3_x_axis: geometry collision mesh filename=comau_meshes/q3_m.stl; visual mesh filename=comau_meshes/q3_m.stl
- link link4_x_axis: geometry collision mesh filename=comau_meshes/q4_m.stl; visual mesh filename=comau_meshes/q4_m.stl
- link link5_x_axis: geometry collision mesh filename=comau_meshes/q5_m.stl; visual mesh filename=comau_meshes/q5_m.stl
- link link6_x_axis: geometry collision mesh filename=comau_meshes/q6_m.stl; visual mesh filename=comau_meshes/q6_m.stl

Commit message: added 3d printing head to comau simulation using custom coupling frame

File: examples/robot_descriptions/comau_NJ290_3-0_m.urdf (robot description, URDF)
Before this commit: robot example_robot, 21 links, 20 joints
Links:
- removed link link6_y_axis
- added link printing_coupling_frame; visual cylinder length=0.2 radius=0.01
Joints:
- joint q6_y: child link6_y_axis -> printing_coupling_frame; origin xyz=0 0 0 rpy=0 1.571 0 -> xyz=0 0 0 rpy=1.571 0 0
