Commit message: updated igus name to follow naming scheme

File: examples/robot_descriptions/igus_4dof_robot.urdf (robot description, URDF)
Before this commit: robot igus_4DOF_SV, 5 links, 4 joints
Links:
- link base_link: geometry collision mesh filename=igus_4dof_robot_meshes/Joint0Coll.dae scale=0.001 0.001 0.001; visual mesh filename=igus_4dof_robot_meshes/Joint0.dae scale=0.001 0.001 0.001
- link link1: geometry collision mesh filename=igus_4dof_robot_meshes/Joint1Coll.dae scale=0.001 0.001 0.001; visual mesh filename=igus_4dof_robot_meshes/Joint1.dae scale=0.001 0.001 0.001
- link link2: geometry collision mesh filename=igus_4dof_robot_meshes/Joint2Coll.dae scale=0.001 0.001 0.001; visual mesh filename=igus_4dof_robot_meshes/Joint2.dae scale=0.001 0.001 0.001
- link link3: geometry collision mesh filename=igus_4dof_robot_meshes/Joint3Coll.dae scale=0.001 0.001 0.001; visual mesh filename=igus_4dof_robot_meshes/Joint3.dae scale=0.001 0.001 0.001
- link link4: geometry collision mesh filename=igus_4dof_robot_meshes/Joint4.dae scale=0.001 0.001 0.001; visual mesh filename=igus_4dof_robot_meshes/Joint4.dae scale=0.001 0.001 0.001
