Commit message: added contact values to screwdriver tcp

File: examples/robot_descriptions/screwDriver.urdf (robot description, URDF)
Before this commit: robot gripper, 2 links, 1 joints
Links:
- link baseLink: geometry visual mesh filename=tool_mesh/base_m.stl
- link tcp: geometry collision cylinder length=0.08 radius=0.01; visual cylinder length=0.08 radius=0.01
