Commit message: latest results
latest resuslts

File: examples/robot_descriptions/comau_nj290_robot.urdf (robot description, URDF)
Before this commit: robot example_robot, 21 links, 20 joints
Joints:
- joint q1: limit lower=-3.14159265358 upper=3.14159265358 effort=204 velocity=1.91986217719 -> (none); type revolute -> continuous

Commit message: update

File: examples/robot_descriptions/comau_nj290_robot.urdf (robot description, URDF)
Before this commit: robot example_robot, 21 links, 20 joints
Joints:
- joint q1: limit (none) -> lower=-3.14159265358 upper=3.14159265358 effort=204 velocity=1.91986217719; type continuous -> revolute
