Commit message: SCARA Robot Setup
- Runnign Setup Scara

File: examples/robot_descriptions/scara_control.urdf (robot description, URDF)
Before this commit: robot scara_control, 4 links, 3 joints
Links:
- link base_link: mass 2.7892 -> None
- link link_1: mass 0.78816 -> None
- link link_2: mass 0.602617398624407 -> None
- link link_3: mass 0.148684285758606 -> None
