Commit message: make_robot_static

File: examples/robot_descriptions/comau_nj290_robotNC.urdf (robot description, URDF)
Before this commit: robot example_robot, 7 links, 6 joints
Joints:
- joint q4: limit lower=-31.4159265358 upper=31.4159265358 effort=204 velocity=1.91986217719 -> lower=-3.14159265358 upper=3.14159265358 effort=204 velocity=1.91986217719
- joint q5: limit lower=-21.816615645 upper=21.816615645 effort=204 velocity=1.91986217719 -> lower=-2.1816615645 upper=2.1816615645 effort=204 velocity=1.91986217719
- joint q6: limit lower=-62.8318530716 upper=62.8318530716 effort=204 velocity=1.91986217719 -> lower=-3.14159265358 upper=3.14159265358 effort=204 velocity=1.91986217719
